File: ayab-silver-reed-shield/ayab-silver-reed-hardware/ayab-silver-reed-hardware.kicad_sch (KiCad schematic)
At the start: 30 parts, among them Q1 2N2222A, Q2 Q_PMOS_GDS, Q3 2N2222A, U1 D3V3XA4B10LP, U2 TLV75801PDRV, U3 ESP32-S3-MINI-1-N8

Commit message: feat: handle ESP32 signals
Parts:
- removed D4: 1N4001, Diode_THT:D_DO-41_SOD81_P10.16mm_Horizontal, symbol Device:D_Small
- added D4: LED, LED_SMD:LED_0603_1608Metric, symbol Device:LED
- added D6: 1N4148WT, Diode_SMD:D_SOD-523, symbol Device:D_Small
- added J1: Conn_01x07_Pin, symbol Connector:Conn_01x07_Pin
- added J5: DIN-7, Locals:DIN-704-M10, symbol symbols:DIN-7
- added J6: Barrel_Jack, Connector_BarrelJack:BarrelJack_Horizontal, symbol Connector:Barrel_Jack
- added R10, R11: 1k, Resistor_SMD:R_0603_1608Metric, symbol Device:R_Small
- added TP1: GND, TestPoint:TestPoint_Pad_D1.0mm, symbol Connector:TestPoint
- added TP2: 16V, TestPoint:TestPoint_Pad_D1.0mm, symbol Connector:TestPoint
- added TP3: 5V, TestPoint:TestPoint_Pad_D1.0mm, symbol Connector:TestPoint
- D2, D3, D5: value 1N4001 -> 1N4148WT; footprint Diode_THT:D_DO-41_SOD81_P10.16mm_Horizontal -> Diode_SMD:D_SOD-523
- F1: footprint (none) -> Capacitor_THT:CP_Radial_D8.0mm_P5.00mm
- Q1, Q3: value 2N2222A -> MMBT2222A; footprint PCM_Package_TO_SOT_THT_AKL:TO-18-3_EBC -> PCM_Package_TO_SOT_SMD_AKL:SOT-23
- R9: value 10k -> 1k
Connections:
- net 16VControlled: now also J5.6, TP2.1
- net 16vIN: now also J6.1, R11.2
- net 3vCCP: now also U3.19 (IO15); no longer U3.16 (IO12)
- net 3vDOB: now also U3.18 (IO14); no longer U3.20 (IO16)
- net 3vHOK: now also U3.16 (IO12); no longer U3.17 (IO13)
- net 3vKSL: now also U3.17 (IO13), D6.2 (A); no longer U3.19 (IO15)
- net 3vND1: now also U3.20 (IO16); no longer U3.18 (IO14)
- net 5VUSB: now also J5.7, R10.1, TP3.1; no longer Q3.3 (C)
- net CCP: now also J1.4 (Pin_4), J5.4
- net GND: now also D4.1 (K), J1.7 (Pin_7), J5.8 (GND), J6.2, TP1.1
- net HOK: now also J1.5 (Pin_5), J5.5
- net ND1: now also J1.1 (Pin_1), J5.1
- net SolenoidControl: now also U3.21 (IO17), J1.6 (Pin_6)
- new net: D4.2 (A), R11.1
- new net DOB: J1.3 (Pin_3), J5.3, Q3.3 (C), R10.2
- new net KSL: D6.1 (K), J1.2 (Pin_2), J5.2
- no-connect marks 35 -> 34
